File: oresat-imu.brd (EAGLE design)
At the start: 100 x 80 mm, 12 parts, among them Q1 CSM-7X-DU, U1 LTC2875XS

Commit message: Added
Parts:
- JP2: device pinhead:1X02 -> pinhead:1X03
Connections:
- new net +5V: JP2.1, JP2.2, JP2.3
- net VCC: no longer JP2.1, JP2.2
Changed lines of the file:
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@@
 <elements>
 <element name="JP1" library="pinhead" package="2X03" value="" x="45.72" y="11.43" rot="R270"/>
-<element name="JP2" library="pinhead" package="1X02" value="" x="41.91" y="2.54"/>
+<element name="JP2" library="pinhead" package="1X03" value="" x="41.91" y="2.54"/>
 <element name="JP3" library="pinhead" package="1X02" value="" x="35.56" y="2.54"/>
 <element name="JP4" library="pinhead" package="1X07" value="" x="52.07" y="44.45"/>
@@
 </signal>
 <signal name="VCC">
-<contactref element="JP2" pad="2"/>
-<contactref element="JP2" pad="1"/>
 <contactref element="U1" pad="3"/>
 <contactref element="U$1" pad="5"/>
@@
 <wire x1="37.78" y1="29.845" x2="41.42" y2="30.08" width="0" layer="19" extent="1-1"/>
 <wire x1="46.99" y1="13.97" x2="52.385" y2="25.4" width="0" layer="19" extent="1-1"/>
-<wire x1="43.18" y1="2.54" x2="46.99" y2="13.97" width="0" layer="19" extent="1-1"/>
-<wire x1="40.64" y1="2.54" x2="43.18" y2="2.54" width="0" layer="19" extent="1-1"/>
-<wire x1="2.54" y1="10.16" x2="40.64" y2="2.54" width="0" layer="19" extent="1-1"/>
+<wire x1="2.54" y1="10.16" x2="37.78" y2="29.845" width="0" layer="19" extent="1-1"/>
 </signal>
 <signal name="DIO1">
@@
 <contactref element="U$1" pad="31"/>
 </signal>
+<signal name="+5V">
+<contactref element="JP2" pad="2"/>
+<contactref element="JP2" pad="1"/>
+<contactref element="JP2" pad="3"/>
+<wire x1="41.91" y1="2.54" x2="44.45" y2="2.54" width="0" layer="19" extent="1-1"/>
+<wire x1="39.37" y1="2.54" x2="41.91" y2="2.54" width="0" layer="19" extent="1-1"/>
+</signal>
 </signals>
