File: oresat-imu.sch (EAGLE design)
At the start: 11 parts, among them Q1 CSM-7X-DU, U1 LTC2875XS

Commit message: Added
Parts:
- added JP6: SUPPLY, pinhead:PINHD-1X2/90
- JP2: device pinhead:PINHD-1X2 -> pinhead:PINHD-1X3
- JP5: value (none) -> CAN
Connections:
- removed net N$1: JP4.1
- removed net N$2: JP4.2
- removed net N$3: JP4.3
- removed net N$4: JP4.4
- removed net N$5: JP4.5
- removed net N$6: JP4.6
- removed net N$7: JP4.7
- new net +5V: JP2.1, JP2.2, JP2.3
- new net ADIS_NRST: JP4.7, U$1.PB0
- new net AUX_ADC: JP4.5, U$1.PB3
- new net AUX_DAC: JP4.6, U$1.PB1
- new net CAN_SLEEP: U$1.PA13, U1.RS1
- new net DIO1: JP4.1, U$1.PB7
- new net DIO2: JP4.2, U$1.PB6
- new net DIO3: JP4.3, U$1.PB5
- new net DIO4/CLKIN: JP4.4, U$1.PB4
- new net N$10: U$1.PB8-BOOT0
- net GND: now also JP6.2
- net VCC: now also JP6.1; no longer JP2.1, JP2.2
Other:
- note added: "NOTE: ADIS SPI 3.3V compatible"
- note added: "TO ADIS16405"
- moved on the sheet: JP1, JP3, JP4, JP5, Q1, U1
